File: HW/jupiter/cpu_rom_ram.sch (KiCad schematic (older format))
At the start: 3 parts, among them U4 WD65C816S_PLCC44-65xx

Commit message: Added PCB train technical capabilities.
Parts:
- C6, C7: footprint Capacitor_THT:C_Disc_D4.7mm_W2.5mm_P5.00mm -> Capacitor_THT:C_Disc_D3.8mm_W2.6mm_P2.50mm
Changed lines of the file:
@@
 F 0 "C7" V 3246 1025 50  0000 C CNN
 F 1 "0.1uF" V 3375 1025 50  0000 C CNN
-F 2 "Capacitor_THT:C_Disc_D4.7mm_W2.5mm_P5.00mm" H 3475 1025 50  0001 C CNN
+F 2 "Capacitor_THT:C_Disc_D3.8mm_W2.6mm_P2.50mm" H 3475 1025 50  0001 C CNN
 F 3 "~" H 3475 1025 50  0001 C CNN
 	1    3475 1025
@@
 F 0 "C6" V 1721 1025 50  0000 C CNN
 F 1 "0.1uF" V 1850 1025 50  0000 C CNN
-F 2 "Capacitor_THT:C_Disc_D4.7mm_W2.5mm_P5.00mm" H 1950 1025 50  0001 C CNN
+F 2 "Capacitor_THT:C_Disc_D3.8mm_W2.6mm_P2.50mm" H 1950 1025 50  0001 C CNN
 F 3 "~" H 1950 1025 50  0001 C CNN
 	1    1950 1025
