File: HW/jupiter/power_glue_expansion.sch (KiCad schematic (older format))
At the start: 28 parts

Commit message: Started PCB. CPU, RTC and support section added.
Parts:
- C1: renamed from C?; footprint (none) -> Capacitor_THT:CP_Radial_Tantal_D4.5mm_P2.50mm
- C2: renamed from C?; footprint (none) -> Capacitor_THT:C_Disc_D4.7mm_W2.5mm_P5.00mm
- C3, C4: renamed from C?; footprint (none) -> Capacitor_THT:CP_Axial_L10.0mm_D4.5mm_P15.00mm_Horizontal
- D1: renamed from D?; footprint (none) -> LED_THT:LED_D3.0mm
- F1, F2: renamed from F?; footprint (none) -> Fuse:Fuseholder_Cylinder-5x20mm_Schurter_0031_8201_Horizontal_Open
- H1, H2, H3, H4, H5, H6: renamed from H?; footprint (none) -> MountingHole:MountingHole_3.2mm_M3_Pad
- J1: renamed from J?; footprint (none) -> Connector_Molex:Molex_Nano-Fit_105313-xx04_1x04_P2.50mm_Horizontal
- Q1: renamed from Q?; footprint (none) -> Package_TO_SOT_THT:TO-92_HandSolder
- R1, R2, R3, R4: renamed from R?; footprint (none) -> Resistor_THT:R_Axial_DIN0207_L6.3mm_D2.5mm_P7.62mm_Horizontal
- SW1, SW2: renamed from SW?; footprint (none) -> Button_Switch_THT:SW_PUSH_6mm_H4.3mm
- SW3: renamed from SW?; footprint (none) -> Grotto:SW-SPDT-0900766b81587629
- U1: renamed from U?; footprint (none) -> Package_DIP:DIP-8_W7.62mm_Socket
- U2: renamed from U?; footprint (none) -> Package_DIP:DIP-14_W7.62mm_Socket
- gave numbers to parts that had none: 2
Connections:
- net VCC: now also Q1.2 (B)

Commit message: Added PCB train technical capabilities.
Parts:
- C3, C4: footprint Capacitor_THT:CP_Axial_L10.0mm_D4.5mm_P15.00mm_Horizontal -> Capacitor_THT:CP_Radial_D6.3mm_P2.50mm
- Q1: footprint Package_TO_SOT_THT:TO-92_HandSolder -> Package_TO_SOT_THT:TO-92_Inline
Changed lines of the file:
@@
 F 0 "Q1" H 4166 5254 50  0000 L CNN
 F 1 "DS1813" H 3675 5475 50  0000 L CNN
-F 2 "Package_TO_SOT_THT:TO-92_HandSolder" H 4175 5400 50  0001 C CNN
+F 2 "Package_TO_SOT_THT:TO-92_Inline" H 4175 5400 50  0001 C CNN
 F 3 "~" H 3975 5300 50  0001 C CNN
 	1    3975 5300
@@
 F 0 "C3" H 6625 5775 50  0000 L CNN
 F 1 "100uF" H 6625 5625 50  0000 L CNN
-F 2 "Capacitor_THT:CP_Axial_L10.0mm_D4.5mm_P15.00mm_Horizontal" H 6625 5700 50  0001 C CNN
+F 2 "Capacitor_THT:CP_Radial_D6.3mm_P2.50mm" H 6625 5700 50  0001 C CNN
 F 3 "~" H 6625 5700 50  0001 C CNN
 	1    6625 5700
@@
 F 0 "C4" H 8025 5525 50  0000 L CNN
 F 1 "100uF" H 8025 5375 50  0000 L CNN
-F 2 "Capacitor_THT:CP_Axial_L10.0mm_D4.5mm_P15.00mm_Horizontal" H 7975 5450 50  0001 C CNN
+F 2 "Capacitor_THT:CP_Radial_D6.3mm_P2.50mm" H 7975 5450 50  0001 C CNN
 F 3 "~" H 7975 5450 50  0001 C CNN
 	1    7975 5450
